Commit message: added trajectory

File: spirits_description/config/spirits.config.xacro (robot description, xacro)
@@ -1,10 +1,12 @@
 <?xml version="1.0"?>
 <!-- spirits manipulator -->
-<robot xmlns:xacro="http://www.ros.org/wiki/xacro" name="spirits">
+<robot xmlns:xacro="http://www.ros.org/wiki/xacro" name="spirits2">
     <!-- Import spirits urdf file -->
     <xacro:include filename="$(find spirits_description)/urdf/spirits.urdf" />
     <!-- Import spirits ros2_control description -->
+    <xacro:include filename="$(find spirits_description)/urdf/inchworm.urdf" />
+    <!-- Import spirits ros2_control description -->
     <xacro:include filename="$(find spirits_description)/ros2_control/spirits.ros2_control.urdf" />
     <!-- Import all Gazebo-customization elements -->
-    <xacro:include filename="$(find spirits_description)/gazebo/spirits.gazebo.xacro"/>
+    <!-- <xacro:include filename="$(find spirits_description)/gazebo/spirits.gazebo.xacro"/> -->
 </robot>

File: spirits_description/urdf/spirits.urdf (robot description, URDF)
Before this commit: robot spirits, 7 links, 6 joints
Links:
- removed link inchworm
- removed link needle
- removed link tool0
- link base_link: geometry collision mesh filename=package://spirits_description/meshes/bw_base.dae scale=0.001 0.001 0.001; visual mesh filename=package://spirits_description/meshes/bw_base_color.dae scale=0.001 0.001 0.001
- link link1: geometry collision mesh filename=package://spirits_description/meshes/bras_1.dae scale=0.001 0.001 0.001; visual mesh filename=package://spirits_description/meshes/bras_1_color.dae scale=0.001 0.001 0.001
- link link2: geometry collision mesh filename=package://spirits_description/meshes/bras_2.dae scale=0.001 0.001 0.001; visual mesh filename=package://spirits_description/meshes/bras_2_color.dae scale=0.001 0.001 0.001
Joints:
- removed joint joint3
- removed joint needle2inchworm
- removed joint tool02needle
- joint joint1: limit lower=-0.5 upper=0.5 effort=1 velocity=4.8 -> lower=-0.6 upper=0.6 effort=1 velocity=4.8
- joint joint2: limit lower=-0.5 upper=0.5 effort=1 velocity=4.8 -> lower=-0.8 upper=0.8 effort=1 velocity=4.8
